Commit message: formated

File: robots/hexacopter_uam_description/urdf/hexacopter_uam.urdf (robot description, URDF)
Before this commit: robot aerial_manipulator_urdf, 4 links, 3 joints
Links:
- added link arm_link3, mass 0.
Joints:
- added joint arm_link2_arm_link3: type fixed, parent arm_link2, child arm_link3, origin xyz=0 0 0.14 rpy=0 0 0, axis 0 0 0, limit lower=0 upper=0 effort=0 velocity=0
