Commit message: Renaming to match hexarotor structure

File: robots/hexarotor_680_description/urdf/hexarotor_680_flying_arm_2.urdf (robot description, URDF)
Before this commit: robot aerial_manipulator_urdf, 5 links, 4 joints
Links:
- link arm_base_link: geometry collision mesh filename=package://example-robot-data/robots/hexarotor_680_descripti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; visual mesh filename=package://example-robot-data/robots/hexarotor_680_descripti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
- link arm_link1: geometry collision mesh filename=package://example-robot-data/robots/hexarotor_680_descripti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; visual mesh filename=package://example-robot-data/robots/hexarotor_680_descripti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
- link arm_link2: geometry collision mesh filename=package://example-robot-data/robots/hexarotor_680_descripti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; visual mesh filename=package://example-robot-data/robots/hexarotor_680_descripti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
- link base_link: geometry collision mesh filename=package://example-robot-data/robots/hexarotor_680_descripti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; visual mesh filename=package://example-robot-data/robots/hexarotor_680_descripti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
