Commit message: Updated models

File: robots/hexarotor_370_description/urdf/hexarotor_370_flying_arm_3.urdf (robot description, URDF)
Before this commit: robot hexarotor_370_flying_arm_3, 5 links, 4 joints
Links:
- added link arm_link3, mass 0.030904; collision mesh filename=package://example-robot-data/robots/flying_arm_3_descriptio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; visual mesh filename=package://example-robot-data/robots/flying_arm_3_descriptio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
- link arm_ee: mass 0.030904 -> 0.; geometry 
Joints:
- removed joint arm_link2_ee
- added joint arm_link2_arm_link3: type revolute, parent arm_link2, child arm_link3, origin xyz=0.075 0 0 rpy=0 0 0, axis 0 0 1, limit lower=-1.9 upper=1.9 effort=0 velocity=3
- added joint arm_link3_ee: type fixed, parent arm_link3, child arm_ee, origin xyz=0.05 0 -0.015 rpy=0 0 0, axis 0 0 0, limit lower=0 upper=0 effort=0 velocity=0
- joint arm_bl_link1: limit lower=0 upper=0 effort=0 velocity=0 -> lower=-1.9 upper=1.9 effort=0 velocity=3
- joint arm_link1_link2: limit lower=0 upper=0 effort=0 velocity=0 -> lower=-1.9 upper=1.9 effort=0 velocity=3
