Commit message: Flyin arm 3 added

File: robots/flying_arm_5_description/urdf/flying_arm_5.urdf (robot description, URDF)
Before this commit: robot urdf, 6 links, 5 joints
Links:
- link arm_baselink: geometry collision mesh filename=package://example-robot-data/robots/flying_arm_5_descriptio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; visual mesh filename=package://example-robot-data/robots/flying_arm_5_descriptio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
- link arm_ee: geometry collision mesh filename=package://example-robot-data/robots/flying_arm_5_descriptio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; visual mesh filename=package://example-robot-data/robots/flying_arm_5_descriptio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
- link arm_link1: geometry collision mesh filename=package://example-robot-data/robots/flying_arm_5_descriptio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; visual mesh filename=package://example-robot-data/robots/flying_arm_5_descriptio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
- link arm_link2: geometry collision mesh filename=package://example-robot-data/robots/flying_arm_5_descriptio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; visual mesh filename=package://example-robot-data/robots/flying_arm_5_descriptio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
- link arm_link3: geometry collision mesh filename=package://example-robot-data/robots/flying_arm_5_descriptio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; visual mesh filename=package://example-robot-data/robots/flying_arm_5_descriptio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
- link arm_link4: geometry collision mesh filename=package://example-robot-data/robots/flying_arm_5_descriptio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; visual mesh filename=package://example-robot-data/robots/flying_arm_5_descriptio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

Commit message: Renewed Hexacopter370

File: robots/flying_arm_5_description/urdf/flying_arm_5.urdf (robot description, URDF)
Before this commit: robot flying_arm_5, 6 links, 5 joints
Links:
- added link world
Joints:
- added joint fixed: type fixed, parent world, child arm_baselink

File: robots/iris_description/robots/iris_simple.urdf (robot description, URDF)
Before this commit: robot iris, 6 links, 5 joints
Links:
- removed link iris__/imu_link
- removed link iris__base_link
- removed link iris__rotor_0
- removed link iris__rotor_1
- removed link iris__rotor_2
- removed link iris__rotor_3
- added link base_link, mass 1.5; collision box size=0.47 0.47 0.11; visual mesh filename=package://example-robot-data/robots/iris_description/meshes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 scale=1 1 1
- added link rotor_0, mass 0.005; collision cylinder length=0.005 radius=0.128; visual mesh filename=package://example-robot-data/robots/iris_description/meshes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 scale=1 1 1
- added link rotor_1, mass 0.005; collision cylinder length=0.005 radius=0.128; visual mesh filename=package://example-robot-data/robots/iris_description/meshes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 scale=1 1 1
- added link rotor_2, mass 0.005; collision cylinder length=0.005 radius=0.128; visual mesh filename=package://example-robot-data/robots/iris_description/meshes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 scale=1 1 1
- added link rotor_3, mass 0.005; collision cylinder length=0.005 radius=0.128; visual mesh filename=package://example-robot-data/robots/iris_description/meshes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 scale=1 1 1
Joints:
- removed joint iris__/imu_joint
- removed joint iris__rotor_0_joint
- removed joint iris__rotor_1_joint
- removed joint iris__rotor_2_joint
- removed joint iris__rotor_3_joint
- added joint rotor_0_joint: type fixed, parent base_link, child rotor_0, origin xyz=0.13  -0.22   0.023 rpy=0  0  0
- added joint rotor_1_joint: type fixed, parent base_link, child rotor_1, origin xyz=-0.13   0.2    0.023 rpy=0  0  0
- added joint rotor_2_joint: type fixed, parent base_link, child rotor_2, origin xyz=0.13   0.22   0.023 rpy=0  0  0
- added joint rotor_3_joint: type fixed, parent base_link, child rotor_3, origin xyz=-0.13  -0.2    0.023 rpy=0  0  0
