Commit message: Iris standarized

File: robots/iris_description/robots/iris.urdf (robot description, URDF)
Before this commit: robot iris, 6 links, 5 joints
Links:
- removed link iris__/imu_link
Joints:
- removed joint iris__/imu_joint
- joint iris__rotor_0_joint: axis 0  0  1 -> (none); limit lower=-1e+16 upper=1e+16 effort=0.0 velocity=0.0 -> (none); type revolute -> fixed
- joint iris__rotor_1_joint: axis 0  0  1 -> (none); limit lower=-1e+16 upper=1e+16 effort=0.0 velocity=0.0 -> (none); type revolute -> fixed
- joint iris__rotor_2_joint: axis 0  0  1 -> (none); limit lower=-1e+16 upper=1e+16 effort=0.0 velocity=0.0 -> (none); type revolute -> fixed
- joint iris__rotor_3_joint: axis 0  0  1 -> (none); limit lower=-1e+16 upper=1e+16 effort=0.0 velocity=0.0 -> (none); type revolute -> fixed
