Commit message: [hexacopter370_flying_arm_3] added gripper

File: robots/hexacopter370_description/urdf/hexacopter370_flying_arm_3.urdf (robot description, URDF)
Before this commit: robot hexacopter370_flying_arm_3, 11 links, 10 joints
Links:
- added link flying_arm_3__gripper, mass 0.0
Joints:
- added joint flying_arm_3__j_link_3_gripper: type fixed, parent flying_arm_3__link_3, child flying_arm_3__gripper, origin xyz=0.05 0 -0.01 rpy=0 0 0, axis 0 0 1
