Commit message: [feature] addition of TiltHex

File: robots/hextilt_description/urdf/hextilt_flying_arm_5.urdf (robot description, URDF)
Before this commit: robot tilt_hex_flying_arm_5.urdf, 7 links, 6 joints
Links:
- removed link arm_baselink
- removed link arm_ee
- removed link arm_link1
- removed link arm_link2
- removed link arm_link3
- removed link arm_link4
- removed link base_link
- added link flying_arm_5__base_link, mass 0.27973; collision mesh filename=package://example-robot-data/robots/flying_arm_5_descriptio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; visual mesh filename=package://example-robot-data/robots/flying_arm_5_descriptio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
- added link flying_arm_5__gripper, mass 0.0
- added link flying_arm_5__link_1, mass 0.12284; collision mesh filename=package://example-robot-data/robots/flying_arm_5_descriptio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; visual mesh filename=package://example-robot-data/robots/flying_arm_5_descriptio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
- added link flying_arm_5__link_2, mass 0.11474; collision mesh filename=package://example-robot-data/robots/flying_arm_5_descriptio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; visual mesh filename=package://example-robot-data/robots/flying_arm_5_descriptio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
- added link flying_arm_5__link_3, mass 0.068772; collision mesh filename=package://example-robot-data/robots/flying_arm_5_descriptio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; visual mesh filename=package://example-robot-data/robots/flying_arm_5_descriptio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
- added link flying_arm_5__link_4, mass 0.05914; collision mesh filename=package://example-robot-data/robots/flying_arm_5_descriptio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; visual mesh filename=package://example-robot-data/robots/flying_arm_5_descriptio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
- added link flying_arm_5__link_5, mass 0.021791; collision mesh filename=package://example-robot-data/robots/flying_arm_5_descriptio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; visual mesh filename=package://example-robot-data/robots/flying_arm_5_descriptio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
- added link hextilt__base_link, mass 1.0194; collision mesh filename=package://example-robot-data/robots/hextilt_description/mes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; visual mesh filename=package://example-robot-data/robots/hextilt_description/mes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
Joints:
- removed joint arm_bl_link1
- removed joint arm_link1_link2
- removed joint arm_link2_link3
- removed joint arm_link3_link4
- removed joint arm_link4_ee
- removed joint base_link_arm_bl
- added joint flying_arm_5__j_base_link: type fixed, parent hextilt__base_link, child flying_arm_5__base_link, origin xyz=0.0 0 -0.0516 rpy=0 0 0, axis 0 0 0
- added joint flying_arm_5__j_base_link_link_1: type revolute, parent flying_arm_5__base_link, child flying_arm_5__link_1, origin xyz=0 0 0 rpy=1.5708 1.5708 0, axis 0 0 1, limit lower=-1.6707963267948966 upper=1.6707963267948966 effort=1 velocity=10000
- added joint flying_arm_5__j_link_1_link_2: type revolute, parent flying_arm_5__link_1, child flying_arm_5__link_2, origin xyz=0.132 0 0 rpy=0 0 0, axis 0 0 1, limit lower=-1.6707963267948966 upper=1.6707963267948966 effort=1 velocity=10000
- added joint flying_arm_5__j_link_2_link_3: type revolute, parent flying_arm_5__link_2, child flying_arm_5__link_3, origin xyz=0.075 0 0 rpy=0 0 0, axis 0 0 1, limit lower=-1.6707963267948966 upper=1.6707963267948966 effort=0.3 velocity=10000
- added joint flying_arm_5__j_link_3_link_4: type revolute, parent flying_arm_5__link_3, child flying_arm_5__link_4, origin xyz=0 0 -0.011925 rpy=1.5708 0 0, axis 0 0 1, limit lower=-1.6707963267948966 upper=1.6707963267948966 effort=0.3 velocity=10000
- added joint flying_arm_5__j_link_4_link_5: type revolute, parent flying_arm_5__link_4, child flying_arm_5__link_5, origin xyz=0.034 0 -0.00025 rpy=1.5708 0 1.5708, axis 0 0 1, limit lower=-1.6707963267948966 upper=1.6707963267948966 effort=0.3 velocity=10000
- added joint flying_arm_5__j_link_5_gripper: type fixed, parent flying_arm_5__link_5, child flying_arm_5__gripper, origin xyz=0.00 0 0.06 rpy=0 0 0, axis 0 0 1

File: robots/iris_description/robots/iris.urdf (robot description, URDF)
Before this commit: robot iris, 5 links, 4 joints
Links:
- removed link iris__rotor_0
- removed link iris__rotor_1
- removed link iris__rotor_2
- removed link iris__rotor_3
Joints:
- removed joint iris__rotor_0_joint
- removed joint iris__rotor_1_joint
- removed joint iris__rotor_2_joint
- removed joint iris__rotor_3_joint
