Commit message: [robots] hexacopter680 added

File: robots/hexacopter680_description/urdf/hexacopter680_flying_arm_2.urdf (robot description, URDF)
Before this commit: robot hexarotor_680_description, 5 links, 4 joints
Links:
- removed link arm_base_link
- removed link arm_link1
- removed link arm_link2
- removed link arm_link3
- removed link base_link
- added link flying_arm_2__base_link, mass 0.23972; collision mesh filename=package://example-robot-data/robots/hexacopter680_descripti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; visual mesh filename=package://example-robot-data/robots/hexacopter680_descripti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
- added link flying_arm_2__gripper, mass 0.
- added link flying_arm_2__link_1, mass 0.077411; collision mesh filename=package://example-robot-data/robots/hexacopter680_descripti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; visual mesh filename=package://example-robot-data/robots/hexacopter680_descripti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
- added link flying_arm_2__link_2, mass 0.16984; collision mesh filename=package://example-robot-data/robots/hexacopter680_descripti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; visual mesh filename=package://example-robot-data/robots/hexacopter680_descripti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
- added link hexacopter680__base_link, mass 2.8968; collision mesh filename=package://example-robot-data/robots/hexacopter680_descripti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; visual mesh filename=package://example-robot-data/robots/hexacopter680_descripti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
Joints:
- removed joint arm_base_link_arm_link1
- removed joint arm_link1_arm_link2
- removed joint arm_link2_arm_link3
- removed joint base_link_arm_base_link
- added joint flying_arm_2__j_base_link: type fixed, parent hexacopter680__base_link, child flying_arm_2__base_link, origin xyz=0.20335 0 -0.0867 rpy=1.5708 0 -1.5708, axis 0 0 0
- added joint flying_arm_2__j_base_link_link_1: type revolute, parent flying_arm_2__base_link, child flying_arm_2__link_1, origin xyz=0 0 0 rpy=1.5708 0 3.1416, axis 1 0 0, limit lower=-1.6707963267948966 upper=1.6707963267948966 effort=1 velocity=10000
- added joint flying_arm_2__j_link_1_link_2: type revolute, parent flying_arm_2__link_1, child flying_arm_2__link_2, origin xyz=0 0 -0.132 rpy=3.1416 0 -3.1416, axis 1 0 0, limit lower=-1.6707963267948966 upper=1.6707963267948966 effort=1 velocity=10000
- added joint flying_arm_3__j_link_2_gripper: type fixed, parent flying_arm_2__link_2, child flying_arm_2__gripper, origin xyz=0 0 0.14 rpy=0 0 0, axis 0 0 0, limit lower=0 upper=0 effort=0 velocity=0
